Commit message: Will now loop between pick, place, and home. Uses PID as control"

File: src/robot_controller/urdf/robot.urdf (robot description, URDF)
Before this commit: robot RRR_arm, 4 links, 3 joints
Links:
- link link1: geometry collision cylinder length=0.2 radius=0.05; visual cylinder length=0.2 radius=0.05
Joints:
- joint joint2: origin xyz=0 0 0.3 rpy=0 0 0 -> xyz=0 0 0.2 rpy=0 0 0

Commit message: now actually pathfinds. also you can enable the visualization of the spheres it uses to check for collisions. I still want to optimize the path that it takes

File: src/robot_controller/urdf/robot.urdf (robot description, URDF)
Before this commit: robot RRR_arm, 4 links, 3 joints
Joints:
- joint joint2: limit lower=-1.57 upper=1.57 effort=10.0 velocity=1.0 -> lower=-3.14 upper=3.14 effort=10.0 velocity=1.0
- joint joint3: limit lower=-1.57 upper=1.57 effort=10.0 velocity=1.0 -> lower=-3.14 upper=3.14 effort=10.0 velocity=1.0
